Commit message: added moveit configurations

File: src/arm/px100_description/urdf/px100.urdf.xacro (robot description, xacro)
@@ -3,11 +3,8 @@
   <xacro:arg name="robot_name" default = "px100"/>
   <xacro:arg name="base_link_frame" default="base_link"/>
-  <xacro:arg name="show_ar_tag" default="false"/>
   <xacro:arg name="show_gripper_bar" default="true"/>
   <xacro:arg name="show_gripper_fingers" default="true"/>
   <xacro:arg name="use_world_frame" default="false"/>
-  <xacro:arg name="external_urdf_loc" default=""/>
   <xacro:arg name="load_gazebo_configs" default="false"/>
-  <xacro:property name="urdf_loc" value="$(arg external_urdf_loc)"/>
   <xacro:property name="pi_offset" value="0.00001"/>
   <xacro:if value="$(arg load_gazebo_configs)">
@@ -241,33 +238,4 @@
     </inertial>
   </link>
-  <!-- If the AR tag is being used, then add the AR tag mount -->
-  <xacro:if value="$(arg show_ar_tag)">
-    <joint name="ar_tag" type="fixed">
-      <axis xyz="0 0 0"/>
-      <origin rpy="0 0 0" xyz="-0.017 0 0.04155"/>
-      <parent link="$(arg robot_name)/ee_arm_link"/>
-      <child link="$(arg robot_name)/ar_tag_link"/>
-    </joint>
-    <link name="$(arg robot_name)/ar_tag_link">
-      <visual>
-        <origin rpy="0 0 0" xyz="0 0 0"/>
-        <geometry>
-          <mesh filename="package://px100_description/meshes/px100_meshes/px100_9_ar_tag.stl" scale="0.001 0.001 0.001"/>
-        </geometry>
-        <material name="px100_black"/>
-      </visual>
-      <collision>
-        <origin rpy="0 0 0" xyz="0 0 0"/>
-        <geometry>
-          <mesh filename="package://px100_description/meshes/px100_meshes/px100_9_ar_tag.stl" scale="0.001 0.001 0.001"/>
-        </geometry>
-      </collision>
-      <inertial>
-        <origin rpy="0 0 0" xyz="0 0 -0.00315"/>
-        <mass value="0.016507"/>
-        <inertia ixx="0.000003084" ixy="0" ixz="0" iyy="0.000003084" iyz="0" izz="0.000006059"/>
-      </inertial>
-    </link>
-  </xacro:if>
   <!-- If the gripper bar is being used, then also add the gripper bar -->
   <xacro:if value="$(arg show_gripper_bar)">
@@ -403,6 +371,3 @@
     </xacro:if>
   </xacro:if>
-  <xacro:if value="${urdf_loc != ''}">
-    <xacro:include filename="${urdf_loc}"/>
-  </xacro:if>
 </robot>

Commit message: added hardware_interface and dynamixel interface

File: src/arm/px100_description/urdf/px100.urdf.xacro (robot description, xacro)
@@ -3,8 +3,11 @@
   <xacro:arg name="robot_name" default = "px100"/>
   <xacro:arg name="base_link_frame" default="base_link"/>
+  <xacro:arg name="show_ar_tag" default="false"/>
   <xacro:arg name="show_gripper_bar" default="true"/>
   <xacro:arg name="show_gripper_fingers" default="true"/>
   <xacro:arg name="use_world_frame" default="false"/>
+  <xacro:arg name="external_urdf_loc" default=""/>
   <xacro:arg name="load_gazebo_configs" default="false"/>
+  <xacro:property name="urdf_loc" value="$(arg external_urdf_loc)"/>
   <xacro:property name="pi_offset" value="0.00001"/>
   <xacro:if value="$(arg load_gazebo_configs)">
@@ -238,4 +241,33 @@
     </inertial>
   </link>
+  <!-- If the AR tag is being used, then add the AR tag mount -->
+  <xacro:if value="$(arg show_ar_tag)">
+    <joint name="ar_tag" type="fixed">
+      <axis xyz="0 0 0"/>
+      <origin rpy="0 0 0" xyz="-0.017 0 0.04155"/>
+      <parent link="$(arg robot_name)/ee_arm_link"/>
+      <child link="$(arg robot_name)/ar_tag_link"/>
+    </joint>
+    <link name="$(arg robot_name)/ar_tag_link">
+      <visual>
+        <origin rpy="0 0 0" xyz="0 0 0"/>
+        <geometry>
+          <mesh filename="package://px100_description/meshes/px100_meshes/px100_9_ar_tag.stl" scale="0.001 0.001 0.001"/>
+        </geometry>
+        <material name="px100_black"/>
+      </visual>
+      <collision>
+        <origin rpy="0 0 0" xyz="0 0 0"/>
+        <geometry>
+          <mesh filename="package://px100_description/meshes/px100_meshes/px100_9_ar_tag.stl" scale="0.001 0.001 0.001"/>
+        </geometry>
+      </collision>
+      <inertial>
+        <origin rpy="0 0 0" xyz="0 0 -0.00315"/>
+        <mass value="0.016507"/>
+        <inertia ixx="0.000003084" ixy="0" ixz="0" iyy="0.000003084" iyz="0" izz="0.000006059"/>
+      </inertial>
+    </link>
+  </xacro:if>
   <!-- If the gripper bar is being used, then also add the gripper bar -->
   <xacro:if value="$(arg show_gripper_bar)">
@@ -371,3 +403,6 @@
     </xacro:if>
   </xacro:if>
+  <xacro:if value="${urdf_loc != ''}">
+    <xacro:include filename="${urdf_loc}"/>
+  </xacro:if>
 </robot>
